Commit message: add p3d plugins and depth camera for aliengo

File: robots/aliengo_description/xacro/gazebo.xacro (robot description, xacro)
@@ -17,4 +17,16 @@
                 <material>Gazebo/Yellow</material>
             </plot>
+        </plugin>
+    </gazebo>
+    <gazebo>
+        <plugin filename="libgazebo_ros_p3d.so" name="p3d_base_controller">
+            <alwaysOn>true</alwaysOn>
+            <updateRate>1000.0</updateRate>
+            <frameName>map</frameName>
+            <bodyName>base</bodyName>
+            <topicName>/odom/ground_truth</topicName>
+            <gaussianNoise>0.00</gaussianNoise>
+            <xyzOffsets>0 0 0</xyzOffsets>
+            <rpyOffsets>0 0 0</rpyOffsets>
         </plugin>
     </gazebo>

File: robots/aliengo_description/xacro/robot.xacro (robot description, xacro)
@@ -5,4 +5,11 @@
     <xacro:include filename="$(find aliengo_description)/xacro/leg.xacro"/>
     <xacro:include filename="$(find aliengo_description)/xacro/gazebo.xacro"/>
+    <xacro:include filename="$(find aliengo_description)/xacro/depthCamera.xacro"/>
+    <xacro:depthCamera camID="1" name="face">
+        <origin rpy="0 ${PI/9} 0" xyz="0.35 0.0 0.15"/>
+    </xacro:depthCamera>
+        <xacro:depthCamera camID="2" name="rear">
+        <origin rpy="0 ${PI/18} ${PI}" xyz="-0.45 0.0 0.15"/>
+    </xacro:depthCamera>
     <!-- Rotor related joint and link is only for demonstrate location. -->
     <!-- Actually, the rotor will rotate and the joint is not fixed. Reduction ratio should be considered. -->
